Commit message: Trying to run demo_gazebo.launch

File: motoman_hc10_moveit_config/urdf/cell.xacro (robot description, xacro)
@@ -5,5 +5,5 @@
       <origin rpy="0 0 0" xyz="0 0 0"/>
       <geometry>
-        <mesh filename="/home/felix/catkin_ws_mm/src/ros_yaskawa_hc10/motoman_hc10_support/meshes/env/pieds_cellule.stl" scale="1 1 1"/>
+        <mesh filename="/home/yaska/catkin_ws/src/ros_yaskawa_hc10/motoman_hc10_support/meshes/env/pieds_cellule.stl" scale="1 1 1"/>
       </geometry>
       <material name="silver"/>
@@ -12,5 +12,5 @@
       <origin rpy="0 0 0" xyz="0 0 0"/>
       <geometry>
-        <mesh filename="home/felix/catkin_ws_mm/src/ros_yaskawa_hc10/motoman_hc10_support/meshes/env/pieds_cellule.stl" scale="1 1 1"/>
+        <mesh filename="home/yaska/catkin_ws/src/ros_yaskawa_hc10/motoman_hc10_support/meshes/env/pieds_cellule.stl" scale="1 1 1"/>
       </geometry>
     </collision>
@@ -20,5 +20,5 @@
       <origin rpy="0 0 0" xyz="0 0 0"/>
       <geometry>
-        <mesh filename="home/felix/catkin_ws_mm/src/ros_yaskawa_hc10/motoman_hc10_support/meshes/env/ergots.stl" scale="0.001 0.001 0.001"/>
+        <mesh filename="home/yaska/catkin_ws/src/ros_yaskawa_hc10/motoman_hc10_support/meshes/env/ergots.stl" scale="0.001 0.001 0.001"/>
       </geometry>
       <material name="dark_gray"/>
@@ -27,5 +27,5 @@
       <origin rpy="0 0 0" xyz="0 0 0"/>
       <geometry>
-        <mesh filename="home/felix/catkin_ws_mm/src/ros_yaskawa_hc10/motoman_hc10_support/meshes/env/ergots.stl" scale="0.001 0.001 0.001"/>
+        <mesh filename="home/yaska/catkin_ws/src/ros_yaskawa_hc10/motoman_hc10_support/meshes/env/ergots.stl" scale="0.001 0.001 0.001"/>
       </geometry>
     </collision>
@@ -35,5 +35,5 @@
       <origin rpy="0 0 0" xyz="0 0 0"/>
       <geometry>
-        <mesh filename="home/felix/catkin_ws_mm/src/ros_yaskawa_hc10/motoman_hc10_support/meshes/env/ergots.stl" scale="0.001 0.001 0.001"/>
+        <mesh filename="home/yaska/catkin_ws/src/ros_yaskawa_hc10/motoman_hc10_support/meshes/env/ergots.stl" scale="0.001 0.001 0.001"/>
       </geometry>
       <material name="dark_gray"/>
@@ -42,5 +42,5 @@
       <origin rpy="0 0 0" xyz="0 0 0"/>
       <geometry>
-        <mesh filename="home/felix/catkin_ws_mm/src/ros_yaskawa_hc10/motoman_hc10_support/meshes/env/ergots.stl" scale="0.001 0.001 0.001"/>
+        <mesh filename="home/yaska/catkin_ws/src/ros_yaskawa_hc10/motoman_hc10_support/meshes/env/ergots.stl" scale="0.001 0.001 0.001"/>
       </geometry>
     </collision>
@@ -50,5 +50,5 @@
       <origin rpy="0 0 0" xyz="0 0 0"/>
       <geometry>
-        <mesh filename="home/felix/catkin_ws_mm/src/ros_yaskawa_hc10/motoman_hc10_support/meshes/env/rail_milieu.stl" scale="0.001 0.001 0.001"/>
+        <mesh filename="home/yaska/catkin_ws/src/ros_yaskawa_hc10/motoman_hc10_support/meshes/env/rail_milieu.stl" scale="0.001 0.001 0.001"/>
       </geometry>
       <material name="silver"/>
@@ -57,5 +57,5 @@
       <origin rpy="0 0 0" xyz="0 0 0"/>
       <geometry>
-        <mesh filename="home/felix/catkin_ws_mm/src/ros_yaskawa_hc10/motoman_hc10_support/meshes/env/rail_milieu.stl" scale="0.001 0.001 0.001"/>
+        <mesh filename="home/yaska/catkin_ws/src/ros_yaskawa_hc10/motoman_hc10_support/meshes/env/rail_milieu.stl" scale="0.001 0.001 0.001"/>
       </geometry>
     </collision>
@@ -65,5 +65,5 @@
       <origin rpy="0 0 0" xyz="0 0 0"/>
       <geometry>
-        <mesh filename="home/felix/catkin_ws_mm/src/ros_yaskawa_hc10/motoman_hc10_support/meshes/env/rail_tournant.stl" scale="0.001 0.001 0.001"/>
+        <mesh filename="home/yaska/catkin_ws/src/ros_yaskawa_hc10/motoman_hc10_support/meshes/env/rail_tournant.stl" scale="0.001 0.001 0.001"/>
       </geometry>
       <material name="silver"/>
@@ -72,5 +72,5 @@
       <origin rpy="0 0 0" xyz="0 0 0"/>
       <geometry>
-        <mesh filename="home/felix/catkin_ws_mm/src/ros_yaskawa_hc10/motoman_hc10_support/meshes/env/rail_tournant.stl" scale="0.001 0.001 0.001"/>
+        <mesh filename="home/yaska/catkin_ws/src/ros_yaskawa_hc10/motoman_hc10_support/meshes/env/rail_tournant.stl" scale="0.001 0.001 0.001"/>
       </geometry>
     </collision>
@@ -80,5 +80,5 @@
       <origin rpy="0 0 0" xyz="0 0 0"/>
       <geometry>
-        <mesh filename="home/felix/catkin_ws_mm/src/ros_yaskawa_hc10/motoman_hc10_support/meshes/env/rail_tournant.stl" scale="0.001 0.001 0.001"/>
+        <mesh filename="home/yaska/catkin_ws/src/ros_yaskawa_hc10/motoman_hc10_support/meshes/env/rail_tournant.stl" scale="0.001 0.001 0.001"/>
       </geometry>
       <material name="silver"/>
@@ -87,5 +87,5 @@
       <origin rpy="0 0 0" xyz="0 0 0"/>
       <geometry>
-        <mesh filename="home/felix/catkin_ws_mm/src/ros_yaskawa_hc10/motoman_hc10_support/meshes/env/rail_tournant.stl" scale="0.001 0.001 0.001"/>
+        <mesh filename="home/yaska/catkin_ws/src/ros_yaskawa_hc10/motoman_hc10_support/meshes/env/rail_tournant.stl" scale="0.001 0.001 0.001"/>
       </geometry>
     </collision>

File: motoman_hc10_moveit_config/urdf/hc10.urdf (robot description, URDF)
Before this commit: robot motoman_hc10, 8 links, 8 joints
Links:
- link base_link: geometry collision mesh filename=home/yaska/catkin_ws/src/ros_yaskawa_hc10/motoman_hc10_supp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; visual mesh filename=home/yaska/catkin_ws/src/ros_yaskawa_hc10/motoman_hc10_supp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
- link link_1_s: geometry collision mesh filename=home/yaska/catkin_ws/src/ros_yaskawa_hc10/motoman_hc10_supp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; visual mesh filename=home/yaska/catkin_ws/src/ros_yaskawa_hc10/motoman_hc10_supp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
- link link_2_l: geometry collision mesh filename=package://motoman_hc10_support/meshes/hc10/collision/link_2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; visual mesh filename=home/yaska/catkin_ws/src/ros_yaskawa_hc10/motoman_hc10_supp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
- link link_3_u: geometry collision mesh filename=home/yaska/catkin_ws/src/ros_yaskawa_hc10/motoman_hc10_supp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; visual mesh filename=home/yaska/catkin_ws/src/ros_yaskawa_hc10/motoman_hc10_supp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
- link link_4_r: geometry collision mesh filename=home/yaska/catkin_ws/src/ros_yaskawa_hc10/motoman_hc10_supp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; visual mesh filename=home/yaska/catkin_ws/src/ros_yaskawa_hc10/motoman_hc10_supp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
- link link_5_b: geometry collision mesh filename=home/yaska/catkin_ws/src/ros_yaskawa_hc10/motoman_hc10_supp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; visual mesh filename=home/yaska/catkin_ws/src/ros_yaskawa_hc10/motoman_hc10_supp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
- link link_6_t: geometry collision mesh filename=home/yaska/catkin_ws/src/ros_yaskawa_hc10/motoman_hc10_supp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; visual mesh filename=home/yaska/catkin_ws/src/ros_yaskawa_hc10/motoman_hc10_supp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

File: motoman_hc10_moveit_config/urdf/hc10_only.urdf (robot description, URDF)
Before this commit: robot yaskawa_1, 10 links, 9 joints
Links:
- link base_link: geometry collision mesh filename=home/yaska/catkin_ws/src/ros_yaskawa_hc10/motoman_hc10_supp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; visual mesh filename=home/yaska/catkin_ws/src/ros_yaskawa_hc10/motoman_hc10_supp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
- link link_1_s: geometry collision mesh filename=home/yaska/catkin_ws/src/ros_yaskawa_hc10/motoman_hc10_supp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; visual mesh filename=home/yaska/catkin_ws/src/ros_yaskawa_hc10/motoman_hc10_supp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
- link link_2_l: geometry collision mesh filename=home/yaska/catkin_ws/src/ros_yaskawa_hc10/motoman_hc10_supp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; visual mesh filename=home/yaska/catkin_ws/src/ros_yaskawa_hc10/motoman_hc10_supp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
- link link_3_u: geometry collision mesh filename=home/yaska/catkin_ws/src/ros_yaskawa_hc10/motoman_hc10_supp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; visual mesh filename=home/yaska/catkin_ws/src/ros_yaskawa_hc10/motoman_hc10_supp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
- link link_4_r: geometry collision mesh filename=home/yaska/catkin_ws/src/ros_yaskawa_hc10/motoman_hc10_supp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; visual mesh filename=home/yaska/catkin_ws/src/ros_yaskawa_hc10/motoman_hc10_supp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
- link link_5_b: geometry collision mesh filename=home/yaska/catkin_ws/src/ros_yaskawa_hc10/motoman_hc10_supp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; visual mesh filename=home/yaska/catkin_ws/src/ros_yaskawa_hc10/motoman_hc10_supp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
- link link_6_t: geometry collision mesh filename=home/yaska/catkin_ws/src/ros_yaskawa_hc10/motoman_hc10_supp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; visual mesh filename=home/yaska/catkin_ws/src/ros_yaskawa_hc10/motoman_hc10_supp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

File: motoman_hc10_moveit_config/urdf/hc10_with_env.xacro (robot description, xacro)
@@ -2,9 +2,9 @@
 <robot name="yaskawa_1" xmlns:xacro="http://www.ros.org/wiki/xacro" >
     <!-- loading urdf -->
-    <xacro:include filename="home/felix/catkin_ws_mm/src/ros_yaskawa_hc10/motoman_hc10_moveit_config/urdf/materials.xacro" />
-    <xacro:include filename="home/felix/catkin_ws_mm/src/ros_yaskawa_hc10/motoman_hc10_moveit_config/urdf/hc10dt_b10.xacro" />
-    <xacro:include filename="home/felix/catkin_ws_mm/src/ros_yaskawa_hc10/motoman_hc10_moveit_config/urdf/table.xacro" />
-    <xacro:include filename="home/felix/catkin_ws_mm/src/ros_yaskawa_hc10/motoman_hc10_moveit_config/urdf/cell.xacro" />
-    <xacro:include filename="home/felix/catkin_ws_mm/src/ros_yaskawa_hc10/motoman_hc10_moveit_config/urdf/pince.xacro" />
+    <xacro:include filename="home/yaska/catkin_ws/src/ros_yaskawa_hc10/motoman_hc10_moveit_config/urdf/materials.xacro" />
+    <xacro:include filename="home/yaska/catkin_ws/src/ros_yaskawa_hc10/motoman_hc10_moveit_config/urdf/hc10dt_b10.xacro" />
+    <xacro:include filename="home/yaska/catkin_ws/src/ros_yaskawa_hc10/motoman_hc10_moveit_config/urdf/table.xacro" />
+    <xacro:include filename="home/yaska/catkin_ws/src/ros_yaskawa_hc10/motoman_hc10_moveit_config/urdf/cell.xacro" />
+    <xacro:include filename="home/yaska/catkin_ws/src/ros_yaskawa_hc10/motoman_hc10_moveit_config/urdf/pince.xacro" />
     <!-- linking robot to world,workspaces and end-effector -->
     <link name="world" />

File: motoman_hc10_moveit_config/urdf/hc10dt_b10.xacro (robot description, xacro)
@@ -1,5 +1,5 @@
 <?xml version="1.0" ?>
 <robot name="motoman_hc10dt_b10" xmlns:xacro="http://ros.org/wiki/xacro">
-  <xacro:include filename="home/felix/catkin_ws_mm/src/ros_yaskawa_hc10/motoman_hc10_support/urdf/hc10dt_b10_macro.xacro" />
+  <xacro:include filename="home/yaska/catkin_ws/src/ros_yaskawa_hc10/motoman_hc10_support/urdf/hc10dt_b10_macro.xacro" />
   <xacro:motoman_hc10dt_b10 prefix="yaska1_"/>
 </robot>

File: motoman_hc10_moveit_config/urdf/hc10dt_b10_macro.xacro (robot description, xacro)
@@ -2,10 +2,10 @@
 <robot xmlns:xacro="http://ros.org/wiki/xacro">
   <xacro:macro name="motoman_hc10dt_b10" params="prefix">
-    <xacro:include filename="home/felix/catkin_ws_mm/src/ros_yaskawa_hc10/motoman_resources/urdf/common_materials.xacro"/>
+    <xacro:include filename="home/yaska/catkin_ws/src/ros_yaskawa_hc10/motoman_resources/urdf/common_materials.xacro"/>
     <!-- link list -->
     <link name="${prefix}base_link">
       <visual>
         <geometry>
-          <mesh filename="home/felix/catkin_ws_mm/src/ros_yaskawa_hc10/motoman_hc10_support/meshes/hc10dt_b10/visual/base_link.dae"/>
+          <mesh filename="home/yaska/catkin_ws/src/ros_yaskawa_hc10/motoman_hc10_support/meshes/hc10dt_b10/visual/base_link.dae"/>
         </geometry>
         <xacro:material_yaskawa_blue/>
@@ -13,5 +13,5 @@
       <collision>
         <geometry>
-          <mesh filename="home/felix/catkin_ws_mm/src/ros_yaskawa_hc10/motoman_hc10_support/meshes/hc10dt_b10/collision/base_link.stl"/>
+          <mesh filename="home/yaska/catkin_ws/src/ros_yaskawa_hc10/motoman_hc10_support/meshes/hc10dt_b10/collision/base_link.stl"/>
         </geometry>
       </collision>
@@ -20,5 +20,5 @@
       <visual>
         <geometry>
-          <mesh filename="home/felix/catkin_ws_mm/src/ros_yaskawa_hc10/motoman_hc10_support/meshes/hc10dt_b10/visual/link_1_s.dae"/>
+          <mesh filename="home/yaska/catkin_ws/src/ros_yaskawa_hc10/motoman_hc10_support/meshes/hc10dt_b10/visual/link_1_s.dae"/>
         </geometry>
         <xacro:material_yaskawa_blue/>
@@ -26,5 +26,5 @@
       <collision>
         <geometry>
-          <mesh filename="home/felix/catkin_ws_mm/src/ros_yaskawa_hc10/motoman_hc10_support/meshes/hc10dt_b10/collision/link_1_s.stl"/>
+          <mesh filename="home/yaska/catkin_ws/src/ros_yaskawa_hc10/motoman_hc10_support/meshes/hc10dt_b10/collision/link_1_s.stl"/>
         </geometry>
       </collision>
@@ -33,5 +33,5 @@
       <visual>
         <geometry>
-          <mesh filename="home/felix/catkin_ws_mm/src/ros_yaskawa_hc10/motoman_hc10_support/meshes/hc10dt_b10/visual/link_2_l.dae"/>
+          <mesh filename="home/yaska/catkin_ws/src/ros_yaskawa_hc10/motoman_hc10_support/meshes/hc10dt_b10/visual/link_2_l.dae"/>
         </geometry>
         <xacro:material_yaskawa_blue/>
@@ -39,5 +39,5 @@
       <collision>
         <geometry>
-          <mesh filename="home/felix/catkin_ws_mm/src/ros_yaskawa_hc10/motoman_hc10_support/meshes/hc10dt_b10/collision/link_2_l.stl"/>
+          <mesh filename="home/yaska/catkin_ws/src/ros_yaskawa_hc10/motoman_hc10_support/meshes/hc10dt_b10/collision/link_2_l.stl"/>
         </geometry>
       </collision>
@@ -46,5 +46,5 @@
       <visual>
         <geometry>
-          <mesh filename="home/felix/catkin_ws_mm/src/ros_yaskawa_hc10/motoman_hc10_support/meshes/hc10dt_b10/visual/link_3_u.dae"/>
+          <mesh filename="home/yaska/catkin_ws/src/ros_yaskawa_hc10/motoman_hc10_support/meshes/hc10dt_b10/visual/link_3_u.dae"/>
         </geometry>
         <xacro:material_yaskawa_blue/>
@@ -52,5 +52,5 @@
       <collision>
         <geometry>
-          <mesh filename="home/felix/catkin_ws_mm/src/ros_yaskawa_hc10/motoman_hc10_support/meshes/hc10dt_b10/collision/link_3_u.stl"/>
+          <mesh filename="home/yaska/catkin_ws/src/ros_yaskawa_hc10/motoman_hc10_support/meshes/hc10dt_b10/collision/link_3_u.stl"/>
         </geometry>
       </collision>
@@ -59,5 +59,5 @@
       <visual>
         <geometry>
-          <mesh filename="home/felix/catkin_ws_mm/src/ros_yaskawa_hc10/motoman_hc10_support/meshes/hc10dt_b10/visual/link_4_r.dae"/>
+          <mesh filename="home/yaska/catkin_ws/src/ros_yaskawa_hc10/motoman_hc10_support/meshes/hc10dt_b10/visual/link_4_r.dae"/>
         </geometry>
         <xacro:material_yaskawa_blue/>
@@ -65,5 +65,5 @@
       <collision>
         <geometry>
-          <mesh filename="home/felix/catkin_ws_mm/src/ros_yaskawa_hc10/motoman_hc10_support/meshes/hc10dt_b10/collision/link_4_r.stl"/>
+          <mesh filename="home/yaska/catkin_ws/src/ros_yaskawa_hc10/motoman_hc10_support/meshes/hc10dt_b10/collision/link_4_r.stl"/>
         </geometry>
       </collision>
@@ -72,5 +72,5 @@
       <visual>
         <geometry>
-          <mesh filename="home/felix/catkin_ws_mm/src/ros_yaskawa_hc10/motoman_hc10_support/meshes/hc10dt_b10/visual/link_5_b.dae"/>
+          <mesh filename="home/yaska/catkin_ws/src/ros_yaskawa_hc10/motoman_hc10_support/meshes/hc10dt_b10/visual/link_5_b.dae"/>
         </geometry>
         <xacro:material_yaskawa_blue/>
@@ -78,5 +78,5 @@
       <collision>
         <geometry>
-          <mesh filename="home/felix/catkin_ws_mm/src/ros_yaskawa_hc10/motoman_hc10_support/meshes/hc10dt_b10/collision/link_5_b.stl"/>
+          <mesh filename="home/yaska/catkin_ws/src/ros_yaskawa_hc10/motoman_hc10_support/meshes/hc10dt_b10/collision/link_5_b.stl"/>
         </geometry>
       </collision>
@@ -85,5 +85,5 @@
       <visual>
         <geometry>
-          <mesh filename="home/felix/catkin_ws_mm/src/ros_yaskawa_hc10/motoman_hc10_support/meshes/hc10dt_b10/visual/link_6_t.dae"/>
+          <mesh filename="home/yaska/catkin_ws/src/ros_yaskawa_hc10/motoman_hc10_support/meshes/hc10dt_b10/visual/link_6_t.dae"/>
         </geometry>
         <xacro:material_yaskawa_blue/>
@@ -91,5 +91,5 @@
       <collision>
         <geometry>
-          <mesh filename="home/felix/catkin_ws_mm/src/ros_yaskawa_hc10/motoman_hc10_support/meshes/hc10dt_b10/collision/link_6_t.stl"/>
+          <mesh filename="home/yaska/catkin_ws/src/ros_yaskawa_hc10/motoman_hc10_support/meshes/hc10dt_b10/collision/link_6_t.stl"/>
        </geometry>
       </collision>

File: motoman_hc10_moveit_config/urdf/pince.xacro (robot description, xacro)
@@ -5,5 +5,5 @@
       <visual>
         <geometry>
-          <mesh filename="home/felix/catkin_ws_mm/src/ros_yaskawa_hc10/motoman_hc10_support/meshes/hand/LWR50F-17-04-A.stl" scale="0.001 0.001 0.001"/>
+          <mesh filename="home/yaska/catkin_ws/src/ros_yaskawa_hc10/motoman_hc10_support/meshes/hand/LWR50F-17-04-A.stl" scale="0.001 0.001 0.001"/>
         </geometry>
         <material name="dark_gray"/>
@@ -11,5 +11,5 @@
       <collision>
         <geometry>
-          <mesh filename="home/felix/catkin_ws_mm/src/ros_yaskawa_hc10/motoman_hc10_support/meshes/hand/LWR50F-17-04-A.stl" scale="0.001 0.001 0.001"/>
+          <mesh filename="home/yaska/catkin_ws/src/ros_yaskawa_hc10/motoman_hc10_support/meshes/hand/LWR50F-17-04-A.stl" scale="0.001 0.001 0.001"/>
         </geometry>
       </collision>
@@ -18,5 +18,5 @@
       <visual>
         <geometry>
-          <mesh filename="home/felix/catkin_ws_mm/src/ros_yaskawa_hc10/motoman_hc10_support/meshes/hand/end_effector_LWR50L-03-00001-A.stl" scale="0.001 0.001 0.001"/>
+          <mesh filename="home/yaska/catkin_ws/src/ros_yaskawa_hc10/motoman_hc10_support/meshes/hand/end_effector_LWR50L-03-00001-A.stl" scale="0.001 0.001 0.001"/>
         </geometry>
         <material name="white_smoke"/>
@@ -24,5 +24,5 @@
       <collision>
         <geometry>
-          <mesh filename="home/felix/catkin_ws_mm/src/ros_yaskawa_hc10/motoman_hc10_support/meshes/hand/end_effector_LWR50L-03-00001-A.stl" scale="0.001 0.001 0.001"/>
+          <mesh filename="home/yaska/catkin_ws/src/ros_yaskawa_hc10/motoman_hc10_support/meshes/hand/end_effector_LWR50L-03-00001-A.stl" scale="0.001 0.001 0.001"/>
         </geometry>
       </collision>
@@ -31,5 +31,5 @@
         <visual>
           <geometry>
-            <mesh filename="home/felix/catkin_ws_mm/src/ros_yaskawa_hc10/motoman_hc10_support/meshes/hand/mors_for_LWR50L-03-00001-A.stl" scale="0.001 0.001 0.001"/>
+            <mesh filename="home/yaska/catkin_ws/src/ros_yaskawa_hc10/motoman_hc10_support/meshes/hand/mors_for_LWR50L-03-00001-A.stl" scale="0.001 0.001 0.001"/>
           </geometry>
           <material name="silver"/>
@@ -37,5 +37,5 @@
         <collision>
           <geometry>
-            <mesh filename="home/felix/catkin_ws_mm/src/ros_yaskawa_hc10/motoman_hc10_support/meshes/hand/mors_for_LWR50L-03-00001-A.stl" scale="0.001 0.001 0.001"/>
+            <mesh filename="home/yaska/catkin_ws/src/ros_yaskawa_hc10/motoman_hc10_support/meshes/hand/mors_for_LWR50L-03-00001-A.stl" scale="0.001 0.001 0.001"/>
           </geometry>
         </collision>
@@ -44,5 +44,5 @@
         <visual>
           <geometry>
-            <mesh filename="home/felix/catkin_ws_mm/src/ros_yaskawa_hc10/motoman_hc10_support/meshes/hand/mors_for_LWR50L-03-00001-A.stl" scale="0.001 0.001 0.001"/>
+            <mesh filename="home/yaska/catkin_ws/src/ros_yaskawa_hc10/motoman_hc10_support/meshes/hand/mors_for_LWR50L-03-00001-A.stl" scale="0.001 0.001 0.001"/>
           </geometry>
           <material name="silver"/>
@@ -50,5 +50,5 @@
         <collision>
           <geometry>
-            <mesh filename="home/felix/catkin_ws_mm/src/ros_yaskawa_hc10/motoman_hc10_support/meshes/hand/mors_for_LWR50L-03-00001-A.stl" scale="0.001 0.001 0.001"/>
+            <mesh filename="home/yaska/catkin_ws/src/ros_yaskawa_hc10/motoman_hc10_support/meshes/hand/mors_for_LWR50L-03-00001-A.stl" scale="0.001 0.001 0.001"/>
           </geometry>
         </collision>

File: motoman_hc10_moveit_config/urdf/table.xacro (robot description, xacro)
@@ -5,5 +5,5 @@
       <origin rpy="0 0 0" xyz="0 0 0"/>
       <geometry>
-        <mesh filename="home/felix/catkin_ws_mm/src/ros_yaskawa_hc10/motoman_hc10_support/meshes/env/table_yaskawa.stl" scale="1 1 1"/>
+        <mesh filename="home/yaska/catkin_ws/src/ros_yaskawa_hc10/motoman_hc10_support/meshes/env/table_yaskawa.stl" scale="1 1 1"/>
       </geometry>
       <material name="silver"/>
@@ -12,5 +12,5 @@
       <origin rpy="0 0 0" xyz="0 0 0"/>
       <geometry>
-        <mesh filename="home/felix/catkin_ws_mm/src/ros_yaskawa_hc10/motoman_hc10_support/meshes/env/table_yaskawa.stl" scale="1 1 1"/>
+        <mesh filename="home/yaska/catkin_ws/src/ros_yaskawa_hc10/motoman_hc10_support/meshes/env/table_yaskawa.stl" scale="1 1 1"/>
       </geometry>
     </collision>
