Commit message: Trying to run demo_gazebo.launch

File: motoman_hc10_support/urdf/pince.xacro (robot description, xacro)
@@ -5,5 +5,5 @@
       <visual>
         <geometry>
-          <mesh filename="/home/felix/catkin_ws_mm/src/ros_yaskawa_hc10/motoman_hc10_support/meshes/hand/LWR50F-17-04-A.stl" scale="0.001 0.001 0.001"/>
+          <mesh filename="/home/yaska/catkin_ws/src/ros_yaskawa_hc10/motoman_hc10_support/meshes/hand/LWR50F-17-04-A.stl" scale="0.001 0.001 0.001"/>
         </geometry>
         <material name="dark_gray"/>
@@ -11,5 +11,5 @@
       <collision>
         <geometry>
-          <mesh filename="/home/felix/catkin_ws_mm/src/ros_yaskawa_hc10/motoman_hc10_support/meshes/hand/LWR50F-17-04-A.stl" scale="0.001 0.001 0.001"/>
+          <mesh filename="/home/yaska/catkin_ws/src/ros_yaskawa_hc10/motoman_hc10_support/meshes/hand/LWR50F-17-04-A.stl" scale="0.001 0.001 0.001"/>
         </geometry>
       </collision>
@@ -18,5 +18,5 @@
       <visual>
         <geometry>
-          <mesh filename="/home/felix/catkin_ws_mm/src/ros_yaskawa_hc10/motoman_hc10_support/meshes/hand/end_effector_LWR50L-03-00001-A.stl" scale="0.001 0.001 0.001"/>
+          <mesh filename="/home/yaska/catkin_ws/src/ros_yaskawa_hc10/motoman_hc10_support/meshes/hand/end_effector_LWR50L-03-00001-A.stl" scale="0.001 0.001 0.001"/>
         </geometry>
         <material name="white_smoke"/>
@@ -24,5 +24,5 @@
       <collision>
         <geometry>
-          <mesh filename="/home/felix/catkin_ws_mm/src/ros_yaskawa_hc10/motoman_hc10_support/meshes/hand/end_effector_LWR50L-03-00001-A.stl" scale="0.001 0.001 0.001"/>
+          <mesh filename="/home/yaska/catkin_ws/src/ros_yaskawa_hc10/motoman_hc10_support/meshes/hand/end_effector_LWR50L-03-00001-A.stl" scale="0.001 0.001 0.001"/>
         </geometry>
       </collision>
@@ -31,5 +31,5 @@
         <visual>
           <geometry>
-            <mesh filename="/home/felix/catkin_ws_mm/src/ros_yaskawa_hc10/motoman_hc10_support/meshes/hand/mors_for_LWR50L-03-00001-A.stl" scale="0.001 0.001 0.001"/>
+            <mesh filename="/home/yaska/catkin_ws/src/ros_yaskawa_hc10/motoman_hc10_support/meshes/hand/mors_for_LWR50L-03-00001-A.stl" scale="0.001 0.001 0.001"/>
           </geometry>
           <material name="silver"/>
@@ -37,5 +37,5 @@
         <collision>
           <geometry>
-            <mesh filename="/home/felix/catkin_ws_mm/src/ros_yaskawa_hc10/motoman_hc10_support/meshes/hand/mors_for_LWR50L-03-00001-A.stl" scale="0.001 0.001 0.001"/>
+            <mesh filename="/home/yaska/catkin_ws/src/ros_yaskawa_hc10/motoman_hc10_support/meshes/hand/mors_for_LWR50L-03-00001-A.stl" scale="0.001 0.001 0.001"/>
           </geometry>
         </collision>
@@ -44,5 +44,5 @@
         <visual>
           <geometry>
-            <mesh filename="/home/felix/catkin_ws_mm/src/ros_yaskawa_hc10/motoman_hc10_support/meshes/hand/mors_for_LWR50L-03-00001-A.stl" scale="0.001 0.001 0.001"/>
+            <mesh filename="/home/yaska/catkin_ws/src/ros_yaskawa_hc10/motoman_hc10_support/meshes/hand/mors_for_LWR50L-03-00001-A.stl" scale="0.001 0.001 0.001"/>
           </geometry>
           <material name="silver"/>
@@ -50,5 +50,5 @@
         <collision>
           <geometry>
-            <mesh filename="/home/felix/catkin_ws_mm/src/ros_yaskawa_hc10/motoman_hc10_support/meshes/hand/mors_for_LWR50L-03-00001-A.stl" scale="0.001 0.001 0.001"/>
+            <mesh filename="/home/yaska/catkin_ws/src/ros_yaskawa_hc10/motoman_hc10_support/meshes/hand/mors_for_LWR50L-03-00001-A.stl" scale="0.001 0.001 0.001"/>
           </geometry>
         </collision>

File: motoman_hc10_support/urdf/table.xacro (robot description, xacro)
@@ -5,5 +5,5 @@
       <origin rpy="0 0 0" xyz="0 0 0"/>
       <geometry>
-        <mesh filename="/home/felix/catkin_ws_mm/src/ros_yaskawa_hc10/motoman_hc10_support/meshes/env/table_yaskawa.stl" scale="1 1 1"/>
+        <mesh filename="/home/yaska/catkin_ws/src/ros_yaskawa_hc10/motoman_hc10_support/meshes/env/table_yaskawa.stl" scale="1 1 1"/>
       </geometry>
       <material name="silver"/>
@@ -12,5 +12,5 @@
       <origin rpy="0 0 0" xyz="0 0 0"/>
       <geometry>
-        <mesh filename="/home/felix/catkin_ws_mm/src/ros_yaskawa_hc10/motoman_hc10_support/meshes/env/table_yaskawa.stl" scale="1 1 1"/>
+        <mesh filename="/home/yaska/catkin_ws/src/ros_yaskawa_hc10/motoman_hc10_support/meshes/env/table_yaskawa.stl" scale="1 1 1"/>
       </geometry>
     </collision>

File: motoman_hc10_support/urdf/urdf_new/hc10.urdf (robot description, URDF)
Before this commit: robot motoman_hc10, 8 links, 8 joints
Links:
- link link_3_u: geometry collision mesh filename=home/yaska/catkin_ws/src/ros_yaskawa_hc10/motoman_hc10_supp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; visual mesh filename=package://motoman_hc10_support/meshes/hc10/visual/link_3_u.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

File: motoman_hc10_support/urdf/urdf_new/hc10dt_b10_macro.xacro (robot description, xacro)
@@ -16,4 +16,8 @@
         </geometry>
       </collision>
+        <inertial>
+            <mass value="0.1" />
+            <inertia ixx="0.03" iyy="0.03" izz="0.03" ixy="0.0" ixz="0.0" iyz="0.0" />
+        </inertial>
     </link>
     <link name="${prefix}link_1_s">
@@ -29,4 +33,8 @@
         </geometry>
       </collision>
+        <inertial>
+            <mass value="0.1" />
+            <inertia ixx="0.03" iyy="0.03" izz="0.03" ixy="0.0" ixz="0.0" iyz="0.0" />
+        </inertial>
     </link>
     <link name="${prefix}link_2_l">
@@ -42,4 +50,8 @@
         </geometry>
       </collision>
+        <inertial>
+            <mass value="0.1" />
+            <inertia ixx="0.03" iyy="0.03" izz="0.03" ixy="0.0" ixz="0.0" iyz="0.0" />
+        </inertial>
     </link>
     <link name="${prefix}link_3_u">
@@ -55,4 +67,8 @@
         </geometry>
       </collision>
+        <inertial>
+            <mass value="0.1" />
+            <inertia ixx="0.03" iyy="0.03" izz="0.03" ixy="0.0" ixz="0.0" iyz="0.0" />
+        </inertial>
     </link>
     <link name="${prefix}link_4_r">
@@ -68,4 +84,8 @@
         </geometry>
       </collision>
+        <inertial>
+            <mass value="0.1" />
+            <inertia ixx="0.03" iyy="0.03" izz="0.03" ixy="0.0" ixz="0.0" iyz="0.0" />
+        </inertial>
     </link>
     <link name="${prefix}link_5_b">
@@ -81,4 +101,8 @@
         </geometry>
       </collision>
+        <inertial>
+            <mass value="0.1" />
+            <inertia ixx="0.03" iyy="0.03" izz="0.03" ixy="0.0" ixz="0.0" iyz="0.0" />
+        </inertial>
     </link>
     <link name="${prefix}link_6_t">
@@ -94,4 +118,8 @@
        </geometry>
       </collision>
+        <inertial>
+            <mass value="0.1" />
+            <inertia ixx="0.03" iyy="0.03" izz="0.03" ixy="0.0" ixz="0.0" iyz="0.0" />
+        </inertial>
     </link>
     <!-- end of link list -->
