Commit message: Launch robot in namespace ; separate what needs to be LEFT/RIGHT

File: motoman_hc10_moveit_config/urdf/left/hc10_with_env.xacro (robot description, xacro)
@@ -1,10 +1,11 @@
 <?xml version="1.0" ?>
-<robot name="yaskawa_1" xmlns:xacro="http://www.ros.org/wiki/xacro" >
+<robot name="yaskawa_L" xmlns:xacro="http://www.ros.org/wiki/xacro" >
     <!-- loading urdf -->
     <xacro:include filename="$(find motoman_hc10_moveit_config)/urdf/materials.xacro" />
-    <xacro:include filename="$(find motoman_hc10_moveit_config)/urdf/hc10dt_b10.xacro" />
     <xacro:include filename="$(find motoman_hc10_moveit_config)/urdf/table.xacro" />
-    <xacro:include filename="$(find motoman_hc10_moveit_config)/urdf/cell.xacro" />
-    <xacro:include filename="$(find motoman_hc10_moveit_config)/urdf/pince.xacro" />
+    <xacro:include filename="$(find motoman_hc10_moveit_config)/urdf/left/cell.xacro" />
+    <xacro:include filename="$(find motoman_hc10_moveit_config)/urdf/left/pince.xacro" />
+    <xacro:include filename="$(find motoman_hc10_moveit_config)/urdf/hc10dt_b10_macro.xacro" />
+    <xacro:motoman_hc10dt_b10 prefix=""/>
     <!-- linking robot to world,workspaces and end-effector -->
     <link name="world" />
@@ -14,17 +15,17 @@
         <child link="pieds_cellule_link" />
     </joint>
-    <joint name="world_table" type="fixed">
+    <joint name="world_table_joint" type="fixed">
         <origin rpy="1.57079 0 0" xyz="0 0 0.432"/>
         <parent link="world" />
         <child link="table_link" />
     </joint>
-    <joint name="table_yaska1" type="fixed">
+    <joint name="table_joint" type="fixed">
         <origin rpy="-1.57079 1.57079 0" xyz="0.171 0.203 0.181" />
         <parent link="table_link" />
-        <child link="yaska1_base_link" />
+        <child link="base_link" />
     </joint>
     <joint name="tool_adaptater" type="fixed">
         <origin rpy="-1.57079 0 -1.57079" xyz="0 0 0" />
-        <parent link="yaska1_tool0" />
+        <parent link="tool0" />
         <child link="adaptater_plate_link" />
     </joint>

File: motoman_hc10_moveit_config/urdf/left/pince.xacro (robot description, xacro)
@@ -5,5 +5,5 @@
       <visual>
         <geometry>
-          <mesh filename="package://motoman_hc10_moveit_config/meshes/hand/LWR50F-17-04-A.stl" scale="0.001 0.001 0.001"/>
+          <mesh filename="package://motoman_hc10_moveit_config/meshes/hand/left/LWR50F-17-04-A.stl" scale="0.001 0.001 0.001"/>
         </geometry>
         <material name="dark_gray"/>
@@ -11,5 +11,5 @@
       <collision>
         <geometry>
-          <mesh filename="package://motoman_hc10_moveit_config/meshes/hand/LWR50F-17-04-A.stl" scale="0.001 0.001 0.001"/>
+          <mesh filename="package://motoman_hc10_moveit_config/meshes/hand/left/LWR50F-17-04-A.stl" scale="0.001 0.001 0.001"/>
         </geometry>
       </collision>
@@ -18,5 +18,5 @@
       <visual>
         <geometry>
-          <mesh filename="package://motoman_hc10_moveit_config/meshes/hand/end_effector_LWR50L-03-00001-A.stl" scale="0.001 0.001 0.001"/>
+          <mesh filename="package://motoman_hc10_moveit_config/meshes/hand/left/end_effector_LWR50L-03-00001-A.stl" scale="0.001 0.001 0.001"/>
         </geometry>
         <material name="white_smoke"/>
@@ -24,5 +24,5 @@
       <collision>
         <geometry>
-          <mesh filename="package://motoman_hc10_moveit_config/meshes/hand/end_effector_LWR50L-03-00001-A.stl" scale="0.001 0.001 0.001"/>
+          <mesh filename="package://motoman_hc10_moveit_config/meshes/hand/left/end_effector_LWR50L-03-00001-A.stl" scale="0.001 0.001 0.001"/>
         </geometry>
       </collision>
@@ -31,5 +31,5 @@
         <visual>
           <geometry>
-            <mesh filename="package://motoman_hc10_moveit_config/meshes/hand/mors_for_LWR50L-03-00001-A.stl" scale="0.001 0.001 0.001"/>
+            <mesh filename="package://motoman_hc10_moveit_config/meshes/hand/left/mors_for_LWR50L-03-00001-A.stl" scale="0.001 0.001 0.001"/>
           </geometry>
           <material name="silver"/>
@@ -37,5 +37,5 @@
         <collision>
           <geometry>
-            <mesh filename="package://motoman_hc10_moveit_config/meshes/hand/mors_for_LWR50L-03-00001-A.stl" scale="0.001 0.001 0.001"/>
+            <mesh filename="package://motoman_hc10_moveit_config/meshes/hand/left/mors_for_LWR50L-03-00001-A.stl" scale="0.001 0.001 0.001"/>
           </geometry>
         </collision>
@@ -44,5 +44,5 @@
         <visual>
           <geometry>
-            <mesh filename="package://motoman_hc10_moveit_config/meshes/hand/mors_for_LWR50L-03-00001-A.stl" scale="0.001 0.001 0.001"/>
+            <mesh filename="package://motoman_hc10_moveit_config/meshes/hand/left/mors_for_LWR50L-03-00001-A.stl" scale="0.001 0.001 0.001"/>
           </geometry>
           <material name="silver"/>
@@ -50,5 +50,5 @@
         <collision>
           <geometry>
-            <mesh filename="package://motoman_hc10_moveit_config/meshes/hand/mors_for_LWR50L-03-00001-A.stl" scale="0.001 0.001 0.001"/>
+            <mesh filename="package://motoman_hc10_moveit_config/meshes/hand/left/mors_for_LWR50L-03-00001-A.stl" scale="0.001 0.001 0.001"/>
           </geometry>
         </collision>
@@ -61,5 +61,5 @@
       </joint>
       <!-- ce joint doit être de type prismatique -->
-      <joint name="end_effector_mors1" type="prismatic" >
+      <joint name="end_effector_adaptater_mors1" type="prismatic" >
         <origin rpy="0 0 0" xyz="0 0 0" />
         <parent link="end_effector_link" />

File: motoman_hc10_moveit_config/urdf/right/hc10_with_env.xacro (robot description, xacro)
@@ -1,9 +1,9 @@
 <?xml version="1.0" ?>
-<robot name="yaskawa_L" xmlns:xacro="http://www.ros.org/wiki/xacro" >
+<robot name="yaskawa_R" xmlns:xacro="http://www.ros.org/wiki/xacro" >
     <!-- loading urdf -->
     <xacro:include filename="$(find motoman_hc10_moveit_config)/urdf/materials.xacro" />
     <xacro:include filename="$(find motoman_hc10_moveit_config)/urdf/table.xacro" />
-    <xacro:include filename="$(find motoman_hc10_moveit_config)/urdf/cell.xacro" />
-    <xacro:include filename="$(find motoman_hc10_moveit_config)/urdf/pince.xacro" />
+    <xacro:include filename="$(find motoman_hc10_moveit_config)/urdf/right/cell.xacro" />
+    <xacro:include filename="$(find motoman_hc10_moveit_config)/urdf/right/pince.xacro" />
     <xacro:include filename="$(find motoman_hc10_moveit_config)/urdf/hc10dt_b10_macro.xacro" />
     <xacro:motoman_hc10dt_b10 prefix=""/>
@@ -11,5 +11,5 @@
     <link name="world" />
     <joint name="world_cell" type="fixed">
-        <origin rpy="0 0 -1.57079" xyz="0.72 0.27 0.698"/>
+        <origin rpy="0 0 0" xyz="-0.29 -0.73 0.698"/>
         <parent link="world" />
         <child link="pieds_cellule_link" />
@@ -20,13 +20,13 @@
         <child link="table_link" />
     </joint>
-    <joint name="table_joint" type="fixed">
-        <origin rpy="-1.57079 1.57079 0" xyz="0.171 0.203 0.181" />
+    <joint name="link_base" type="fixed">
+        <origin rpy="-1.57079 3.1415 0" xyz="0.171 0.2 0.181" />
         <parent link="table_link" />
-        <child link="yaskaL_base_link" />
+        <child link="base_link" />
     </joint>
-    <joint name="tool_adaptater" type="fixed">
-        <origin rpy="-1.57079 0 -1.57079" xyz="0 0 0" />
-        <parent link="yaskaL_tool0" />
-        <child link="adaptater_plate_link" />
+    <joint name="tool_cylinder" type="fixed" >
+        <origin rpy="0 0 -1.57079" xyz="0 0 0" />
+        <parent link="tool0" />
+        <child link="cylinder_link" />
     </joint>
 </robot>
