Commit message: fix: use correct model HC10 (NOT DT) for right Yaskawa

File: motoman_hc10_moveit_config/urdf/right/hc10_with_env.xacro (robot description, xacro)
@@ -6,6 +6,6 @@
     <xacro:include filename="$(find motoman_hc10_moveit_config)/urdf/right/cell.xacro" />
     <xacro:include filename="$(find motoman_hc10_moveit_config)/urdf/right/pince.xacro" />
-    <xacro:include filename="$(find motoman_hc10_moveit_config)/urdf/hc10dt_b10_macro.xacro" />
-    <xacro:motoman_hc10dt_b10 prefix=""/>
+    <xacro:include filename="$(find motoman_hc10_support)/urdf/hc10_macro.xacro" />
+    <xacro:motoman_hc10 prefix=""/>
     <!-- linking robot to world,workspaces and end-effector -->
     <link name="world" />
@@ -26,5 +26,5 @@
     </joint>
     <joint name="tool_cylinder" type="fixed" >
-        <origin rpy="0 0 -1.57079" xyz="0 0 0" />
+        <origin rpy="0 0 0" xyz="0 0 0" /> <!-- "0 0 -1.57079"-->
         <parent link="tool0" />
         <child link="cylinder_link" />

Commit message: fix orientation of right-side yaskawa

File: motoman_hc10_moveit_config/urdf/right/hc10_with_env.xacro (robot description, xacro)
@@ -21,5 +21,5 @@
     </joint>
     <joint name="link_base" type="fixed">
-        <origin rpy="-1.57079 3.1415 0" xyz="0.171 0.2 0.181" />
+        <origin rpy="-1.57079 1.57079 0.0" xyz="0.171 0.2 0.181" />
         <parent link="table_link" />
         <child link="base_link" />
